Commit message: 0.3 simple_robot Odometry plugin added

File: simple_robot_description/urdf/wheel.urdf.xacro (robot description, xacro)
@@ -43,5 +43,5 @@
       <turnGravityOff>false</turnGravityOff>
     </gazebo>
-    <joint name="${fb}_${lr}_wheel_joint" type="continuous">
+    <joint name="${fb}_${lr}_joint" type="continuous">
       <parent link="${parent}"/>
       <child link="${fb}_${lr}_wheel"/>
