Commit message: 0.0.7 simple robot This update includes the followings: - A normal distribution added to tick counts - Resolution added to encoder ticks for the motors - A clean xacro with color updates

File: simple_robot_description/urdf/diff_wheeled_robot.xacro (robot description, xacro)
@@ -2,17 +2,4 @@
 <robot name="differential_wheeled_robot" xmlns:xacro="http://www.ros.org/wiki/xacro">
   <xacro:include filename="$(find simple_robot_description)/urdf/wheel.urdf.xacro" />
-  <!-- Defining the colors used in this robot -->
-  <material name="Black">
-    <color rgba="0.0 0.0 0.0 1.0"/>
-  </material>
-  <material name="Red">
-    <color rgba="0.8 0.0 0.0 1.0"/>
-  </material>
-  <material name="White">
-    <color rgba="1.0 1.0 1.0 1.0"/>
-  </material>
-  <material name="Blue">
-    <color rgba="0.0 0.0 0.8 1.0"/>
-  </material>
   <!-- PROPERTY LIST -->
   <!--All units in m-kg-s-radians unit system -->
@@ -127,4 +114,5 @@
         </joint>
         <gazebo reference="caster_front_link">
+          <material>Gazebo/Orange</material>
           <turnGravityOff>false</turnGravityOff>
         </gazebo>
@@ -158,4 +146,5 @@
           </joint>
           <gazebo reference="caster_back_link">
+            <material>Gazebo/Orange</material>
             <turnGravityOff>false</turnGravityOff>
           </gazebo>
@@ -163,27 +152,4 @@
           <wheel fb="front" lr="right" parent="base_link" translateX="0" translateY="0.5" flipY="1"/>
           <wheel fb="front" lr="left" parent="base_link" translateX="0" translateY="-0.5" flipY="1"/>
-          <!-- Differential drive controller  -->
-          <!--<gazebo>
-          <plugin name="differential_drive_controller" filename="libgazebo_ros_diff_drive.so">
-          <rosDebugLevel>Debug</rosDebugLevel>
-          <publishWheelTF>false</publishWheelTF>
-          <robotNamespace>/</robotNamespace>
-          <publishTf>1</publishTf>
-          <publishWheelJointState>false</publishWheelJointState>
-          <alwaysOn>true</alwaysOn>
-          <updateRate>100.0</updateRate>
-          <leftJoint>front_left_wheel_joint</leftJoint>
-          <rightJoint>front_right_wheel_joint</rightJoint>
-          <wheelSeparation>${2*base_radius}</wheelSeparation>
-          <wheelDiameter>${2*wheel_radius}</wheelDiameter>
-          <broadcastTF>1</broadcastTF>
-          <wheelTorque>30</wheelTorque>
-          <wheelAcceleration>1.8</wheelAcceleration>
-          <commandTopic>cmd_vel</commandTopic>
-          <odometryFrame>odom</odometryFrame>
-          <odometryTopic>odom</odometryTopic>
-          <robotBaseFrame>base_footprint</robotBaseFrame>
-        </plugin>
-      </gazebo>-->
       <!-- Bring in simulation data for Gazebo. -->
       <xacro:include filename="$(find simple_robot_description)/urdf/diff_wheeled_robot.gazebo" />

File: simple_robot_description/urdf/wheel.urdf.xacro (robot description, xacro)
@@ -40,5 +40,5 @@
       <kd  value="1.0" />
       <fdir1 value="1 0 0"/>
-      <material>Gazebo/Grey</material>
+      <material>Gazebo/Black</material>
       <turnGravityOff>false</turnGravityOff>
     </gazebo>
@@ -51,13 +51,4 @@
       <joint_properties damping="0.0" friction="0.0"/>
     </joint>
-    <!-- Transmission is important to link the joints and the controller -->
-    <!--<transmission name="${fb}_${lr}_wheel_joint_trans">
-      <type>transmission_interface/SimpleTransmission</type>
-      <joint name="${fb}_${lr}_wheel_joint" />
-      <actuator name="${fb}_${lr}_wheel_joint_motor">
-        <hardwareInterface>EffortJointInterface</hardwareInterface>
-        <mechanicalReduction>1</mechanicalReduction>
-      </actuator>
-    </transmission>-->
   </xacro:macro>
 </robot>
