Commit message: 0.2.2 simple_robot In this update we introduce meshes in gazebo models instead of shape

File: simple_robot_description_4wheels/urdf/robot_4wheels.urdf.xacro (robot description, xacro)
@@ -11,7 +11,7 @@
   <property name="chassis_mass" value="5" /> <!-- in kg-->
   <!-- Wheels -->
-  <xacro:property name="wheel_horizontal_separation" value="0.20" />
-  <xacro:property name="wheel_vertical_separation" value="0.15" />
-  <xacro:property name="wheel_vertical_offset" value="-0.1" />
+  <xacro:property name="wheel_horizontal_separation" value="0.15" />
+  <xacro:property name="wheel_vertical_separation" value="0.23" />
+  <xacro:property name="wheel_vertical_offset" value="-0.13" />
   <xacro:property name="wheel_radius" value="0.098" />
   <xacro:property name="wheel_width" value="0.040" />
@@ -26,5 +26,6 @@
       <origin xyz="0 0 ${footprint_vertical_offset}" rpy="0 0 0"/>
       <geometry>
-        <box size="${chassis_length} ${chassis_width} ${chassis_height}"/>
+	<mesh filename="package://simple_robot_description_4wheels/meshes/inno_sim.stl"/>
+        <!--<box size="${chassis_length} ${chassis_width} ${chassis_height}"/>-->
       </geometry>
       <material name="Black" />

Commit message: 0.2.3 simple_robot In this update we upgrated the move_wheels plugin to support 2wheels and 4wheels

File: simple_robot_description_4wheels/urdf/robot_4wheels.urdf.xacro (robot description, xacro)
@@ -81,5 +81,5 @@
       <material>Gazebo/Red</material>
     </gazebo>
-    <joint name="${prefix}_wheel" type="continuous">
+    <joint name="${prefix}_joint" type="continuous">
       <parent link="chassis_link"/>
       <child link="${prefix}_wheel_link" />

Commit message: 0.2.4 simple_robot In this update we completed the upgrade of the encoders plugin to support 4 wheels and we increase the friction coefficients of the wheels to avoid slipage

File: simple_robot_description_4wheels/urdf/robot_4wheels.urdf.xacro (robot description, xacro)
@@ -29,5 +29,5 @@
         <!--<box size="${chassis_length} ${chassis_width} ${chassis_height}"/>-->
       </geometry>
-      <material name="Black" />
+      <material name="Grey" />
     </visual>
     <collision>
@@ -79,4 +79,6 @@
     </link>
     <gazebo reference="${prefix}_wheel_link">
+      <mu1>100</mu1>
+      <mu2>100</mu2>
       <material>Gazebo/Red</material>
     </gazebo>

Commit message: 0.2.5 simple_robot In this update we upgraded the simple controller to support 2 and 4 wheels. Additionally, we debugged the 4wheels robot (base_footprint)

File: simple_robot_description_4wheels/urdf/robot_4wheels.urdf.xacro (robot description, xacro)
@@ -16,8 +16,27 @@
   <xacro:property name="wheel_radius" value="0.098" />
   <xacro:property name="wheel_width" value="0.040" />
-  <link name="base_link"></link>
+  <!-- BASE-FOOTPRINT -->
+  <!-- base_footprint is a fictitious link(frame) that is on the ground right below base_link origin -->
+  <link name="base_footprint">
+    <inertial>
+      <mass value="0.0001" />
+      <origin xyz="0 0 0" />
+      <inertia ixx="0.0001" ixy="0.0" ixz="0.0"
+        iyy="0.0001" iyz="0.0"
+        izz="0.0001" />
+      </inertial>
+      <visual>
+        <origin xyz="0 0 0" rpy="0 0 0" />
+        <geometry>
+          <box size="0.001 0.001 0.001" />
+        </geometry>
+      </visual>
+    </link>
+    <gazebo reference="base_footprint">
+      <turnGravityOff>false</turnGravityOff>
+    </gazebo>
   <joint name="base_link_joint" type="fixed">
     <origin xyz="0 0 0" rpy="0 0 0" />
-    <parent link="base_link"/>
+    <parent link="base_footprint"/>
     <child link="chassis_link" />
   </joint>
@@ -79,6 +98,6 @@
     </link>
     <gazebo reference="${prefix}_wheel_link">
-      <mu1>100</mu1>
-      <mu2>100</mu2>
+      <!--<mu1>10</mu1>
+      <mu2>10</mu2>-->
       <material>Gazebo/Red</material>
     </gazebo>

Commit message: 0.2.8 simple_robot Laser scanner added to the 4-wheels robot

File: simple_robot_description_4wheels/urdf/robot_4wheels.urdf.xacro (robot description, xacro)
@@ -73,6 +73,6 @@
   <!-- Start of Wheels
   -->
-  <xacro:macro name="wheel" params="prefix *joint_pose">
-  <link name="${prefix}_wheel_link">
+  <xacro:macro name="wheel" params="prefix trans_x trans_y trans_z">
+  <link name="${prefix}_wheel">
     <visual>
       <origin xyz="0 0 0" rpy="${M_PI/2} 0 0"/>
@@ -97,5 +97,5 @@
       </inertial>
     </link>
-    <gazebo reference="${prefix}_wheel_link">
+    <gazebo reference="${prefix}_wheel">
       <!--<mu1>10</mu1>
       <mu2>10</mu2>-->
@@ -104,23 +104,40 @@
     <joint name="${prefix}_joint" type="continuous">
       <parent link="chassis_link"/>
-      <child link="${prefix}_wheel_link" />
-      <xacro:insert_block name="joint_pose" />
+      <child link="${prefix}_wheel" />
+      <origin xyz="${trans_x} ${trans_y} ${trans_z}" rpy="0 0 0" />
       <axis xyz="0 1 0" />
     </joint>
   </xacro:macro>
-  <xacro:wheel prefix="front_left">
-    <origin xyz="${wheel_horizontal_separation} ${wheel_vertical_separation+wheel_width/2} ${wheel_vertical_offset}" rpy="0 0 0" />
-  </xacro:wheel>
-  <xacro:wheel prefix="front_right">
-    <origin xyz="${wheel_horizontal_separation} ${-wheel_vertical_separation-wheel_width/2} ${wheel_vertical_offset}" rpy="0 0 0" />
-  </xacro:wheel>
-  <xacro:wheel prefix="rear_left">
-    <origin xyz="${-wheel_horizontal_separation} ${wheel_vertical_separation+wheel_width/2} ${wheel_vertical_offset}" rpy="0 0 0" />
-  </xacro:wheel>
-  <xacro:wheel prefix="rear_right">
-    <origin xyz="${-wheel_horizontal_separation} ${-wheel_vertical_separation-wheel_width/2} ${wheel_vertical_offset}" rpy="0 0 0" />
-  </xacro:wheel>
+  <xacro:wheel prefix="front_left" trans_x="${wheel_horizontal_separation}" trans_y="${wheel_vertical_separation+wheel_width/2}" trans_z="${wheel_vertical_offset}"/>
+  <xacro:wheel prefix="front_right" trans_x="${wheel_horizontal_separation}" trans_y="${-wheel_vertical_separation-wheel_width/2}" trans_z="${wheel_vertical_offset}"/>
+  <xacro:wheel prefix="rear_left" trans_x="${-wheel_horizontal_separation}" trans_y="${wheel_vertical_separation+wheel_width/2}" trans_z="${wheel_vertical_offset}"/>
+  <xacro:wheel prefix="rear_right" trans_x="${-wheel_horizontal_separation}" trans_y="${-wheel_vertical_separation-wheel_width/2}" trans_z="${wheel_vertical_offset}"/>
   <!-- End of Wheels
   -->
+  <joint name="hokuyo_joint" type="fixed">
+    <origin xyz="0.262 0 0.1" rpy="0 0 0"/>
+    <parent link="chassis_link"/>
+    <child link="hokuyo_link"/>
+  </joint>
+  <!-- Hokuyo Laser -->
+  <link name="hokuyo_link">
+    <collision>
+      <origin xyz="0 0 0" rpy="0 0 0"/>
+      <geometry>
+         <box size="0.1 0.1 0.1"/>
+      </geometry>
+    </collision>
+    <visual>
+      <origin xyz="0 0 0" rpy="0 0 0"/>
+      <geometry>
+        <mesh filename="package://simple_robot_description_2wheels/meshes/hokuyo.dae"/>
+      </geometry>
+    </visual>
+    <inertial>
+      <mass value="1e-5" />
+      <origin xyz="0 0 0" rpy="0 0 0"/>
+      <inertia ixx="1e-6" ixy="0" ixz="0" iyy="1e-6" iyz="0" izz="1e-6" />
+    </inertial>
+  </link>
   <!-- Bring in simulation data for Gazebo. -->
   <xacro:include filename="$(find simple_robot_description_4wheels)/urdf/robot_4wheels.gazebo" />
