Commit message: 0.2.1 simple_robot In this update we have further tidied up the 2wheels and 4wheels models

File: simple_robot_description_2wheels/urdf/diff_wheeled_robot.xacro (robot description, xacro)
@@ -1,5 +1,5 @@
 <?xml version="1.0"?>
 <robot name="differential_wheeled_robot" xmlns:xacro="http://www.ros.org/wiki/xacro">
-  <xacro:include filename="$(find simple_robot_description)/urdf/wheel.urdf.xacro" />
+  <xacro:include filename="$(find simple_robot_description_2wheels)/urdf/wheel.urdf.xacro" />
   <!-- PROPERTY LIST -->
   <!--All units in m-kg-s-radians unit system -->
@@ -153,4 +153,4 @@
           <wheel fb="front" lr="left" parent="base_link" translateX="0" translateY="-0.5" flipY="1"/>
       <!-- Bring in simulation data for Gazebo. -->
-      <xacro:include filename="$(find simple_robot_description)/urdf/diff_wheeled_robot.gazebo" />
+      <xacro:include filename="$(find simple_robot_description_2wheels)/urdf/diff_wheeled_robot.gazebo" />
     </robot>

File: simple_robot_description_4wheels/urdf/robot_4wheels.urdf.xacro (robot description, xacro)
@@ -1,4 +1,4 @@
 <?xml version="1.0"?>
-<robot name="camera_robot" xmlns:xacro="http://www.ros.org/wiki/xacro">
+<robot name="robot" xmlns:xacro="http://www.ros.org/wiki/xacro">
   <!-- PROPERTY LIST -->
   <!--All units in m-kg-s-radians unit system -->
@@ -10,11 +10,4 @@
   <property name="chassis_length" value="0.6" />
   <property name="chassis_mass" value="5" /> <!-- in kg-->
-  <!-- Rotators
-  <xacro:property name="rotator_base" value="0.4" />
-  <xacro:property name="rotator_track" value="0.3" />
-  <xacro:property name="rotator_vertical_offset" value="-0.1" />
-  <xacro:property name="rotator_radius" value="0.025" />
-  <xacro:property name="rotator_width" value="0.08" />
-  -->
   <!-- Wheels -->
   <xacro:property name="wheel_horizontal_separation" value="0.20" />
@@ -109,4 +102,4 @@
   -->
   <!-- Bring in simulation data for Gazebo. -->
-  <xacro:include filename="$(find camera_robot_description)/urdf/camera_robot.gazebo" />
+  <xacro:include filename="$(find simple_robot_description_4wheels)/urdf/robot_4wheels.gazebo" />
 </robot>

Commit message: 0.2.6 simple_robot Laser scanner added to the 2-wheels robot and a labyrinth simple world created

File: simple_robot_description_2wheels/urdf/diff_wheeled_robot.xacro (robot description, xacro)
@@ -152,4 +152,29 @@
           <wheel fb="front" lr="right" parent="base_link" translateX="0" translateY="0.5" flipY="1"/>
           <wheel fb="front" lr="left" parent="base_link" translateX="0" translateY="-0.5" flipY="1"/>
+          <joint name="hokuyo_joint" type="fixed">
+            <origin xyz="0 0 0.04" rpy="0 0 0"/>
+            <parent link="base_link"/>
+            <child link="hokuyo_link"/>
+          </joint> -->
+          <!-- Hokuyo Laser -->
+          <link name="hokuyo_link">
+            <collision>
+              <origin xyz="0 0 0" rpy="0 0 0"/>
+              <geometry>
+        	       <box size="0.1 0.1 0.1"/>
+              </geometry>
+            </collision>
+            <visual>
+              <origin xyz="0 0 0" rpy="0 0 0"/>
+              <geometry>
+                <mesh filename="package://simple_robot_description_2wheels/meshes/hokuyo.dae"/>
+              </geometry>
+            </visual>
+            <inertial>
+              <mass value="1e-5" />
+              <origin xyz="0 0 0" rpy="0 0 0"/>
+              <inertia ixx="1e-6" ixy="0" ixz="0" iyy="1e-6" iyz="0" izz="1e-6" />
+            </inertial>
+          </link>
       <!-- Bring in simulation data for Gazebo. -->
       <xacro:include filename="$(find simple_robot_description_2wheels)/urdf/diff_wheeled_robot.gazebo" />

Commit message: 0.2.5 simple_robot_description_2wheels IMU added to the 2-wheels robot

File: simple_robot_description_2wheels/urdf/diff_wheeled_robot.xacro (robot description, xacro)
@@ -4,33 +4,33 @@
   <!-- PROPERTY LIST -->
   <!--All units in m-kg-s-radians unit system -->
-  <property name="M_PI" value="3.1415926535897931" />
-  <property name="M_PI_2" value="1.570796327" />
-  <property name="DEG_TO_RAD" value="0.017453293" />
+  <xacro:property name="M_PI" value="3.1415926535897931" />
+  <xacro:property name="M_PI_2" value="1.570796327" />
+  <xacro:property name="DEG_TO_RAD" value="0.017453293" />
   <!-- Main body radius and height -->
   <!-- Main Body Cylinder base   -->
-  <property name="base_height" value="0.02" />
-  <property name="base_radius" value="0.15" />
-  <property name="base_mass" value="5" /> <!-- in kg-->
+  <xacro:property name="base_height" value="0.02" />
+  <xacro:property name="base_radius" value="0.15" />
+  <xacro:property name="base_mass" value="5" /> <!-- in kg-->
   <!-- caster wheel radius and height -->
   <!-- caster wheel mass -->
-  <property name="caster_f_height" value="0.04" />
-  <property name="caster_f_radius" value="0.025" />
-  <property name="caster_f_mass" value="0.5" /> <!-- in kg-->
+  <xacro:property name="caster_f_height" value="0.04" />
+  <xacro:property name="caster_f_radius" value="0.025" />
+  <xacro:property name="caster_f_mass" value="0.5" /> <!-- in kg-->
   <!-- caster wheel radius and height -->
   <!-- caster wheel mass -->
-  <property name="caster_b_height" value="0.04" />
-  <property name="caster_b_radius" value="0.025" />
-  <property name="caster_b_mass" value="0.5" /> <!-- in kg-->
+  <xacro:property name="caster_b_height" value="0.04" />
+  <xacro:property name="caster_b_radius" value="0.025" />
+  <xacro:property name="caster_b_mass" value="0.5" /> <!-- in kg-->
   <!-- Wheels -->
-  <property name="wheel_mass" value="2.5" /> --> <!-- in kg-->
-  <property name="base_x_origin_to_wheel_origin" value="0.25" />
-  <property name="base_y_origin_to_wheel_origin" value="0.3" />
-  <property name="base_z_origin_to_wheel_origin" value="0.0" />
+  <xacro:property name="wheel_mass" value="2.5" /> --> <!-- in kg-->
+  <xacro:property name="base_x_origin_to_wheel_origin" value="0.25" />
+  <xacro:property name="base_y_origin_to_wheel_origin" value="0.3" />
+  <xacro:property name="base_z_origin_to_wheel_origin" value="0.0" />
   <!-- Macro for calculating inertia of cylinder -->
-  <macro name="cylinder_inertia" params="m r h">
+  <xacro:macro name="cylinder_inertia" params="m r h">
     <inertia  ixx="${m*(3*r*r+h*h)/12}" ixy = "0" ixz = "0"
       iyy="${m*(3*r*r+h*h)/12}" iyz = "0"
       izz="${m*r*r/2}" />
-    </macro>
+    </xacro:macro>
     <!-- BASE-FOOTPRINT -->
     <!-- base_footprint is a fictitious link(frame) that is on the ground right below base_link origin -->
@@ -162,5 +162,5 @@
               <origin xyz="0 0 0" rpy="0 0 0"/>
               <geometry>
-        	       <box size="0.1 0.1 0.1"/>
+                <box size="0.1 0.1 0.1"/>
               </geometry>
             </collision>
@@ -177,5 +177,16 @@
             </inertial>
           </link>
-      <!-- Bring in simulation data for Gazebo. -->
-      <xacro:include filename="$(find simple_robot_description_2wheels)/urdf/diff_wheeled_robot.gazebo" />
-    </robot>
+          <link name="imu">
+            <inertial>
+              <mass value="0.001"/>
+              <origin xyz="0 0 0" rpy="0 0 0"/>
+              <inertia ixx="1e-6" ixy="0" ixz="0" iyy="1e-6" iyz="0" izz="1e-6" />
+            </inertial>
+          </link>
+          <joint name="imu_joint" type="fixed">
+            <parent link="base_link" />
+            <child link="imu" />
+          </joint>
+          <!-- Bring in simulation data for Gazebo.-->
+          <xacro:include filename="$(find simple_robot_description_2wheels)/urdf/diff_wheeled_robot.gazebo" />
+        </robot>

File: simple_robot_description_2wheels/urdf/wheel.urdf.xacro (robot description, xacro)
@@ -2,15 +2,15 @@
 <robot name="wheel" xmlns:xacro="http://www.ros.org/wiki/xacro">
   <!-- Wheels -->
-  <property name="wheel_radius" value="0.04" />
-  <property name="wheel_height" value="0.02" />
-  <property name="wheel_mass" value="2.5" /> <!-- in kg-->
-  <property name="base_x_origin_to_wheel_origin" value="0.25" />
-  <property name="base_y_origin_to_wheel_origin" value="0.3" />
-  <property name="base_z_origin_to_wheel_origin" value="0.0" />
-  <macro name="cylinder_inertia" params="m r h">
+  <xacro:property name="wheel_radius" value="0.04" />
+  <xacro:property name="wheel_height" value="0.02" />
+  <xacro:property name="wheel_mass" value="2.5" /> <!-- in kg-->
+  <xacro:property name="base_x_origin_to_wheel_origin" value="0.25" />
+  <xacro:property name="base_y_origin_to_wheel_origin" value="0.3" />
+  <xacro:property name="base_z_origin_to_wheel_origin" value="0.0" />
+  <xacro:macro name="cylinder_inertia" params="m r h">
     <inertia  ixx="${m*(3*r*r+h*h)/12}" ixy = "0" ixz = "0"
               iyy="${m*(3*r*r+h*h)/12}" iyz = "0"
               izz="${m*r*r/2}" />
-  </macro>
+  </xacro:macro>
   <xacro:macro name="wheel" params="fb lr parent translateX translateY flipY"> <!--fb : front, back ; lr: left, right -->
     <link name="${fb}_${lr}_wheel">

Commit message: 0.2.6 simple_robot_gazebo (tested only to 2-wheels) - Added a static transform between the EKF frame and the map (ground truth odometry)
0.2.6 simple_robot_description_2wheels
- Housekeeping

0.2.7 simple_robot_description_2wheels
- Fixed the IMU proper functionality after adding the EKF node

0.2.7 simple_robot_control
- Housekeeping; remove unsupported waypoint controller

1.14.4 robot_pose_ekf
- robot_pose_ekf package added
- Disable the tf broadcast to avoid confict with the original one
- Create a new lanch file to accomodate our needs

File: simple_robot_description_2wheels/urdf/diff_wheeled_robot.xacro (robot description, xacro)
@@ -178,5 +178,5 @@
           </link>
           <!-- Imu -->
-          <link name="imu">
+          <link name="imu_link">
             <inertial>
               <mass value="0.001"/>
@@ -187,7 +187,7 @@
           <joint name="imu_joint" type="fixed">
             <parent link="base_link" />
-            <child link="imu" />
+            <child link="imu_link" />
           </joint>
-          <!-- Bring in simulation data for Gazebo.-->
-          <xacro:include filename="$(find simple_robot_description_2wheels)/urdf/diff_wheeled_robot.gazebo" />
-        </robot>
+    <!-- Bring in simulation data for Gazebo.-->
+    <xacro:include filename="$(find simple_robot_description_2wheels)/urdf/diff_wheeled_robot.gazebo" />
+  </robot>

Commit message: 0.2.10 simple_robot_description_2wheels - second IMU added to simulate a scenario like in SIRCAUR project

File: simple_robot_description_2wheels/urdf/diff_wheeled_robot.xacro (robot description, xacro)
@@ -177,6 +177,13 @@
             </inertial>
           </link>
-          <!-- Imu -->
-          <link name="imu_link">
+          <!-- Imu 1-->
+          <link name="imu_link1">
+            <visual>
+              <origin xyz="0 0 0" rpy="0 0 0"/>
+              <geometry>
+                <box size="0.01 0.01 0.01" />
+              </geometry>
+               <material name="Blue" />
+            </visual>
             <inertial>
               <mass value="0.001"/>
@@ -185,7 +192,36 @@
             </inertial>
           </link>
-          <joint name="imu_joint" type="fixed">
+          <gazebo reference="imu_link1">
+            <material>Gazebo/Blue</material>
+            <turnGravityOff>false</turnGravityOff>
+          </gazebo>
+          <joint name="imu_joint1" type="fixed">
+            <origin xyz="0.135 0 0.01" rpy="0 0 0"/>
             <parent link="base_link" />
-            <child link="imu_link" />
+            <child link="imu_link1" />
+          </joint>
+          <!-- Imu 2-->
+          <link name="imu_link2">
+            <visual>
+              <origin xyz="0 0 0" rpy="0 0 0"/>
+              <geometry>
+                <box size="0.01 0.01 0.01" />
+              </geometry>
+               <material name="Red" />
+            </visual>
+            <inertial>
+              <mass value="0.001"/>
+              <origin xyz="0 0 0" rpy="0 0 0"/>
+              <inertia ixx="1e-6" ixy="0" ixz="0" iyy="1e-6" iyz="0" izz="1e-6" />
+            </inertial>
+          </link>
+          <gazebo reference="imu_link2">
+            <material>Gazebo/Red</material>
+            <turnGravityOff>false</turnGravityOff>
+          </gazebo>
+          <joint name="imu_joint2" type="fixed">
+            <origin xyz="-0.135 0 0.01" rpy="0 0 0"/>
+            <parent link="base_link" />
+            <child link="imu_link2" />
           </joint>
     <!-- Bring in simulation data for Gazebo.-->

Commit message: 0.2.11 simple_robot_description_2wheels In this version we added a stereo vision camera to the 2-wheeled robot model

File: simple_robot_description_2wheels/urdf/diff_wheeled_robot.xacro (robot description, xacro)
@@ -152,10 +152,11 @@
           <wheel fb="front" lr="right" parent="base_link" translateX="0" translateY="0.5" flipY="1"/>
           <wheel fb="front" lr="left" parent="base_link" translateX="0" translateY="-0.5" flipY="1"/>
-          <joint name="hokuyo_joint" type="fixed">
-            <origin xyz="0 0 0.04" rpy="0 0 0"/>
-            <parent link="base_link"/>
-            <child link="hokuyo_link"/>
-          </joint> -->
-          <!-- Hokuyo Laser -->
+            <!--
+            <joint name="hokuyo_joint" type="fixed">
+              <origin xyz="0 0 0.04" rpy="0 0 0"/>
+              <parent link="base_link"/>
+              <child link="hokuyo_link"/>
+            </joint>
+          Hokuyo Laser
           <link name="hokuyo_link">
             <collision>
@@ -176,5 +177,5 @@
               <inertia ixx="1e-6" ixy="0" ixz="0" iyy="1e-6" iyz="0" izz="1e-6" />
             </inertial>
-          </link>
+          </link>-->
           <!-- Imu 1-->
           <link name="imu_link1">
@@ -225,4 +226,60 @@
             <child link="imu_link2" />
           </joint>
+          <!-- Kinect -->
+          <joint name="camera_rgb_joint" type="fixed">
+            <origin xyz="0 0 0.05" rpy="0 0 0"/>
+            <parent link="base_link"/>
+            <child link="camera_rgb_frame" />
+          </joint>
+          <link name="camera_rgb_frame"/>
+          <joint name="camera_rgb_optical_joint" type="fixed">
+            <origin xyz="0 0 0" rpy="${-M_PI/2} 0 ${-M_PI/2}" />
+            <parent link="camera_rgb_frame" />
+            <child link="camera_rgb_optical_frame" />
+          </joint>
+          <link name="camera_rgb_optical_frame"/>
+          <joint name="camera_joint" type="fixed">
+            <origin xyz="-0.031 0 -0.016" rpy="0 0 0"/>
+            <parent link="camera_rgb_frame"/>
+            <child link="camera_link"/>
+          </joint>
+          <link name="camera_link">
+            <visual>
+              <origin xyz="0 0 0" rpy="0 0 ${M_PI/2}"/>
+              <geometry>
+                <mesh filename="package://simple_robot_description_2wheels/meshes/kinect.dae"/>
+              </geometry>
+            </visual>
+            <collision>
+              <origin xyz="0.0 0.0 0.0" rpy="0 0 0"/>
+              <geometry>
+                <box size="0.07271 0.27794 0.073"/>
+              </geometry>
+            </collision>
+            <inertial>
+              <mass value="0.564" />
+              <origin xyz="0 0 0" />
+              <inertia ixx="0.003881243" ixy="0.0" ixz="0.0"
+                       iyy="0.000498940" iyz="0.0"
+                       izz="0.003879257" />
+            </inertial>
+          </link>
+          <!-- The fixed joints & links below are usually published by static_transformers launched by the OpenNi launch
+               files. However, for Gazebo simulation we need them, so we add them here.
+               (Hence, don't publish them additionally!) -->
+          <joint name="camera_depth_joint" type="fixed">
+            <origin xyz="0 0 0" rpy="0 0 0" />
+            <parent link="camera_rgb_frame" />
+            <child link="camera_depth_frame" />
+          </joint>
+          <link name="camera_depth_frame"/>
+          <joint name="camera_depth_optical_joint" type="fixed">
+            <origin xyz="0 0 0" rpy="${-M_PI/2} 0 ${-M_PI/2}" />
+            <parent link="camera_depth_frame" />
+            <child link="camera_depth_optical_frame" />
+          </joint>
+          <link name="camera_depth_optical_frame"/>
+    <!-- Kinect sensor for simulation
+    <turtlebot_sim_3dsensor/> -->
     <!-- Bring in simulation data for Gazebo.-->
     <xacro:include filename="$(find simple_robot_description_2wheels)/urdf/diff_wheeled_robot.gazebo" />
